File: RGB LED Driver.brd (EAGLE design)
At the start: 99.1 x 52.1 mm, 11 parts, among them IC1 SN74LS244N, J1 691311400105, J2 691311400102, J3 691311400105

Commit message: Add files via upload
Parts:
- moved W1 3.81 mm to (86.1, 40.0)
- moved J1 1.27 mm to (74.9, 66.0)
- moved J3 1.27 mm to (34.3, 66.0)
Routing:
- net N$19: track 69.7 -> 49.7 mm
- net D6: track 65.3 -> 46.1 mm
- net N$11: track 23.9 -> 41.9 mm
- net N$16: track 72.4 -> 54.8 mm
- net D2: track 74.2 -> 57.3 mm, vias 0 -> 1
- net N$15: track 75.9 -> 59.8 mm
- net D5: track 63.4 -> 48.6 mm
- net +5V: track 106.3 -> 120.9 mm
- net N$20: track 56.5 -> 44.6 mm
- net D4: track 57.6 -> 69.0 mm
- net D8: track 40.7 -> 51.7 mm
- net D3: track 66.4 -> 75.1 mm
- net GND: track 236.3 -> 239.9 mm, vias 1 -> 0
- net N$9: track 17.2 -> 20.8 mm
- net N$10: track 30.2 -> 33.0 mm
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Other:
- outline, holes or cut-outs redrawn
- board text added: "+5"
- board text removed: "+"
